File: electronics/scratch/LED Indicators/LED Indicators.kicad_sch (KiCad schematic)
At the start: 28 parts, among them J1 POWER INPUT, J2 VLOW TP, J3 VHIGH TP, J4 EXTERNAL LED, J5 EXTERNAL TP, SW1 TS-1187A-B-A-B, SW2 TS-1088-AR02016, SW3 SSSS213202, SW4 TS-1088-AR02016, U5 XL-1608UBC-06A, U6 XL-1608PGC-06

Commit message: Finished LED indicator sch, need to run traces next
Parts:
- added JP10, JP8, JP9: SolderJumper_2_Bridged, Jumper:SolderJumper-2_P1.3mm_Bridged_RoundedPad1.0x1.5mm, symbol Jumper:SolderJumper_2_Bridged
- added LED1: P2-0603W6YS2-06T-002, easyeda2kicad:LED-SMD_L1.6-W0.8-RD-WHITE-2, symbol easyeda2kicad:F.0603.00048_P2-0603W6YS2-06T-002
- added LED2: BL-HJC36G-AV-TRB, easyeda2kicad:LED0603-R-RD_AMBER, symbol easyeda2kicad:BL-HJC36G-AV-TRB
- added LED3: CT-1608DUPC-P6, easyeda2kicad:LED-SMD_L1.6-W0.8-RD_CT-1608UWC-P4, symbol easyeda2kicad:CT-1608DUPC-P6
- J1, J2, J3, J4, J5: now not fitted; now left out of the parts list
Connections:
- net +VHIGH: now also JP10.1 (A), JP8.1 (A)
- net +VLOW: now also JP9.1 (A)
- net GND: now also LED1.1 (K), LED2.1 (C), LED3.1 (C)
- new net: JP9.2 (B), LED2.2 (A)
- new net: JP8.2 (B), LED1.2 (A)
- new net: JP10.2 (B), LED3.2 (A)
Other:
- note added: "BRTLED"
- note added: "CHONGTIAN"
- moved on the sheet: JP7, LED11, SW4

Commit message: LED indicators board sent to PCBWay for review
Parts:
- R1: LCSC Part (none) -> C17724
- TP1, TP2: now not fitted; now left out of the parts list
Changed lines of the file:
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@@
 			)
 		)
+		(property "LCSC Part" "C17724"
+			(at 41.91 86.36 90)
+			(hide yes)
+			(show_name no)
+			(do_not_autoplace no)
+			(effects
+				(font
+					(size 1.27 1.27)
+				)
+			)
+		)
 		(pin "1"
 		)
@@
 		(body_style 1)
 		(exclude_from_sim no)
-		(in_bom yes)
+		(in_bom no)
 		(on_board yes)
 		(in_pos_files yes)
-		(dnp no)
+		(dnp yes)
 		(property "Reference" "TP1"
 			(at 32.766 76.454 0)
@@
 		(body_style 1)
 		(exclude_from_sim no)
-		(in_bom yes)
+		(in_bom no)
 		(on_board yes)
 		(in_pos_files yes)
-		(dnp no)
+		(dnp yes)
 		(property "Reference" "TP2"
 			(at 74.93 45.466 0)
