File: electronics/scratch/Pico RP2350 USB Power/Pico RP2350 USB Power.kicad_sch (KiCad schematic)
At the start: 48 parts, among them J1 RFM69HCW, J10 IR TX AOE, J11 IR RX 1, J12 IR RX 2, J13 IR RX 3, J14 BUTTON A, J15 BUTTON B, J16 LED STRIP 1, J17 LED STRIP 2, J18 LED STRIP 3, J19 LED STRIP 4, J2 SD CARD, J20 LED STRIP 5, J21 LED STRIP 6, J22 POWER, J3 I2C_1, J4 I2C_2, J5 I2C_3, J6 STEMMA, J7 I2S AMP, J8 IR TX LINE, J9 IR TX CONE, Q1 AO3406, Q2 AO3406, Q3 AO3406, Q4 AO3401A, Q5 C20917, SW1 POWER, U1 74HCT244

Commit message: L shaped neopixel pin layout
Parts:
- removed SW1: POWER, Button_Switch_THT:SW_DIP_SPSTx01_Slide_9.78x4.72mm_W7.62mm_P2.54mm, symbol Switch:SW_SPST
Other:
- moved on the sheet: J22
Changed lines of the file:
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@@
 	)
 	(junction
-		(at 184.15 133.35)
-		(diameter 0)
-		(color 0 0 0 0)
-	)
-	(junction
 		(at 261.62 148.59)
 		(diameter 0)
@@
 	)
 	(junction
-		(at 199.39 133.35)
-		(diameter 0)
-		(color 0 0 0 0)
-	)
-	(junction
 		(at 191.77 62.23)
 		(diameter 0)
@@
 	(wire
 		(pts
-			(xy 199.39 133.35) (xy 204.47 133.35)
-		)
-		(stroke
-			(width 0)
-			(type default)
-		)
-	)
-	(wire
-		(pts
 			(xy 115.57 99.06) (xy 125.73 99.06)
 		)
@@
 	(wire
 		(pts
-			(xy 184.15 137.16) (xy 184.15 133.35)
-		)
-		(stroke
-			(width 0)
-			(type default)
-		)
-	)
-	(wire
-		(pts
 			(xy 33.02 187.96) (xy 33.02 189.23)
 		)
@@
 	(wire
 		(pts
-			(xy 184.15 133.35) (xy 176.53 133.35)
+			(xy 176.53 133.35) (xy 190.5 133.35)
 		)
 		(stroke
@@
 	(wire
 		(pts
-			(xy 193.04 137.16) (xy 199.39 137.16)
+			(xy 193.04 133.35) (xy 204.47 133.35)
 		)
 		(stroke
@@
 	(wire
 		(pts
-			(xy 196.85 133.35) (xy 199.39 133.35)
-		)
-		(stroke
-			(width 0)
-			(type default)
-		)
-	)
-	(wire
-		(pts
-			(xy 190.5 137.16) (xy 184.15 137.16)
-		)
-		(stroke
-			(width 0)
-			(type default)
-		)
-	)
-	(wire
-		(pts
 			(xy 207.01 25.4) (xy 209.55 25.4)
 		)
@@
 	(wire
 		(pts
-			(xy 186.69 133.35) (xy 184.15 133.35)
-		)
-		(stroke
-			(width 0)
-			(type default)
-		)
-	)
-	(wire
-		(pts
 			(xy 17.78 80.01) (xy 31.75 80.01)
 		)
@@
 	(wire
 		(pts
-			(xy 199.39 137.16) (xy 199.39 133.35)
-		)
-		(stroke
-			(width 0)
-			(type default)
-		)
-	)
-	(wire
-		(pts
 			(xy 26.67 158.75) (xy 26.67 160.02)
 		)
@@
 	(symbol
 		(lib_id "Connector:Conn_01x02_Pin")
-		(at 193.04 142.24 270)
+		(at 193.04 138.43 270)
 		(mirror x)
 		(unit 1)
@@
 		(dnp yes)
 		(property "Reference" "J22"
-			(at 194.818 148.082 90)
+			(at 194.818 144.272 90)
 			(show_name no)
 			(do_not_autoplace no)
@@
 		)
 		(property "Value" "POWER"
-			(at 194.818 145.542 90)
+			(at 194.818 141.732 90)
 			(show_name no)
 			(do_not_autoplace no)
@@
 		)
 		(property "Footprint" "Connector_PinHeader_2.54mm:PinHeader_1x02_P2.54mm_Vertical"
-			(at 193.04 142.24 0)
+			(at 193.04 138.43 0)
 			(hide yes)
 			(show_name no)
@@
 		)
 		(property "Datasheet" ""
-			(at 193.04 142.24 0)
+			(at 193.04 138.43 0)
 			(hide yes)
 			(show_name no)
@@
 		)
 		(property "Description" "Generic connector, single row, 01x02, script generated"
-			(at 193.04 142.24 0)
+			(at 193.04 138.43 0)
 			(hide yes)
 			(show_name no)
@@
 					(unit 1)
 				)
-			)
-		)
-	)
-	(symbol
-		(lib_id "Switch:SW_SPST")
-		(at 191.77 133.35 0)
-		(unit 1)
-		(body_style 1)
-		(exclude_from_sim no)
-		(in_bom no)
-		(on_board yes)
-		(in_pos_files yes)
-		(dnp yes)
-		(fields_autoplaced yes)
-		(property "Reference" "SW1"
-			(at 191.77 127 0)
-			(show_name no)
-			(do_not_autoplace no)
-			(effects
-				(font
-					(size 1.27 1.27)
-				)
-			)
-		)
-		(property "Value" "POWER"
-			(at 191.77 129.54 0)
-			(show_name no)
-			(do_not_autoplace no)
-			(effects
-				(font
-					(size 1.27 1.27)
-				)
-			)
-		)
-		(property "Footprint" "Button_Switch_THT:SW_DIP_SPSTx01_Slide_9.78x4.72mm_W7.62mm_P2.54mm"
-			(at 191.77 133.35 0)
-			(hide yes)
-			(show_name no)
-			(do_not_autoplace no)
-			(effects
-				(font
-					(size 1.27 1.27)
-				)
-			)
-		)
-		(property "Datasheet" ""
-			(at 191.77 133.35 0)
-			(hide yes)
-			(show_name no)
-			(do_not_autoplace no)
-			(effects
-				(font
-					(size 1.27 1.27)
-				)
-			)
-		)
-		(property "Description" "Single Pole Single Throw (SPST) switch"
-			(at 191.77 133.35 0)
-			(hide yes)
-			(show_name no)
-			(do_not_autoplace no)
-			(effects
-				(font
-					(size 1.27 1.27)
-				)
-			)
-		)
-		(pin "2"
-		)
-		(pin "1"
-		)
-		(instances
-			(project "Pico RP2350 USB Power"
-				(path "/f607a6cb-1f81-4ea5-ae65-67dd06ab9fb6"
-					(reference "SW1")
-					(unit 1)
-				)

Commit message: Ground and 3.3v traces, board complete (I think)
Connections:
- net GNDA is gone; now on net GND: A1.33 (AGND)
Changed lines of the file:
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@@
 	(wire
 		(pts
+			(xy 82.55 101.6) (xy 92.71 101.6)
+		)
+		(stroke
+			(width 0)
+			(type default)
+		)
+	)
+	(wire
+		(pts
 			(xy 241.3 22.86) (xy 241.3 24.13)
 		)
@@
 	)
 	(symbol
+		(lib_id "power:GNDA")
+		(at 92.71 101.6 0)
+		(unit 1)
+		(body_style 1)
+		(exclude_from_sim no)
+		(in_bom yes)
+		(on_board yes)
+		(in_pos_files yes)
+		(dnp no)
+		(fields_autoplaced yes)
+		(property "Reference" "#PWR043"
+			(at 92.71 107.95 0)
+			(hide yes)
+			(show_name no)
+			(do_not_autoplace no)
+			(effects
+				(font
+					(size 1.27 1.27)
+				)
+			)
+		)
+		(property "Value" "GNDA"
+			(at 92.71 106.68 0)
+			(show_name no)
+			(do_not_autoplace no)
+			(effects
+				(font
+					(size 1.27 1.27)
+				)
+			)
+		)
+		(property "Footprint" ""
+			(at 92.71 101.6 0)
+			(hide yes)
+			(show_name no)
+			(do_not_autoplace no)
+			(effects
+				(font
+					(size 1.27 1.27)
+				)
+			)
+		)
+		(property "Datasheet" ""
+			(at 92.71 101.6 0)
+			(hide yes)
+			(show_name no)
+			(do_not_autoplace no)
+			(effects
+				(font
+					(size 1.27 1.27)
+				)
+			)
+		)
+		(property "Description" "Power symbol creates a global label with name \"GNDA\" , analog ground"
+			(at 92.71 101.6 0)
+			(hide yes)
+			(show_name no)
+			(do_not_autoplace no)
+			(effects
+				(font
+					(size 1.27 1.27)
+				)
+			)
+		)
+		(pin "1"
+		)
+		(instances
+			(project "Pico RP2350 USB Power"
+				(path "/f607a6cb-1f81-4ea5-ae65-67dd06ab9fb6"
+					(reference "#PWR043")
+					(unit 1)
+				)
+			)
+		)
+	)
+	(symbol
 		(lib_id "Connector_Generic_MountingPin:Conn_01x04_MountingPin")
 		(at 163.83 90.17 0)
@@
 					(unit 1)
 				)
+			)
+		)
+	)
+	(symbol
+		(lib_id "power:GND")
+		(at 82.55 101.6 0)
+		(unit 1)
+		(body_style 1)
+		(exclude_from_sim no)
+		(in_bom yes)
+		(on_board yes)
+		(in_pos_files yes)
+		(dnp no)
+		(fields_autoplaced yes)
+		(property "Reference" "#PWR044"
+			(at 82.55 107.95 0)
+			(hide yes)
+			(show_name no)
+			(do_not_autoplace no)
+			(effects
+				(font
+					(size 1.27 1.27)
+				)
+			)
+		)
+		(property "Value" "GND"
+			(at 82.55 106.68 0)
+			(show_name no)
+			(do_not_autoplace no)
+			(effects
+				(font
+					(size 1.27 1.27)
+				)
+			)
+		)
+		(property "Footprint" ""
+			(at 82.55 101.6 0)
+			(hide yes)
+			(show_name no)
+			(do_not_autoplace no)
+			(effects
+				(font
+					(size 1.27 1.27)
+				)
+			)
+		)
+		(property "Datasheet" ""
+			(at 82.55 101.6 0)
+			(hide yes)
+			(show_name no)
+			(do_not_autoplace no)
+			(effects
+				(font
+					(size 1.27 1.27)
+				)
+			)
+		)
+		(property "Description" "Power symbol creates a global label with name \"GND\" , ground"
+			(at 82.55 101.6 0)
+			(hide yes)
+			(show_name no)
+			(do_not_autoplace no)
+			(effects
+				(font
+					(size 1.27 1.27)
+				)
+			)
+		)
+		(pin "1"
+		)
+		(instances
+			(project "Pico RP2350 USB Power"
+				(path "/f607a6cb-1f81-4ea5-ae65-67dd06ab9fb6"
+					(reference "#PWR044")
+					(unit 1)
+				)

Commit message: RP2350 final adjustments before JLCPCB run
Changed lines of the file:
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@@
 	(wire
 		(pts
-			(xy 82.55 101.6) (xy 92.71 101.6)
-		)
-		(stroke
-			(width 0)
-			(type default)
-		)
-	)
-	(wire
-		(pts
 			(xy 241.3 22.86) (xy 241.3 24.13)
 		)
@@
 	)
 	(symbol
-		(lib_id "power:GNDA")
-		(at 92.71 101.6 0)
-		(unit 1)
-		(body_style 1)
-		(exclude_from_sim no)
-		(in_bom yes)
-		(on_board yes)
-		(in_pos_files yes)
-		(dnp no)
-		(fields_autoplaced yes)
-		(property "Reference" "#PWR043"
-			(at 92.71 107.95 0)
-			(hide yes)
-			(show_name no)
-			(do_not_autoplace no)
-			(effects
-				(font
-					(size 1.27 1.27)
-				)
-			)
-		)
-		(property "Value" "GNDA"
-			(at 92.71 106.68 0)
-			(show_name no)
-			(do_not_autoplace no)
-			(effects
-				(font
-					(size 1.27 1.27)
-				)
-			)
-		)
-		(property "Footprint" ""
-			(at 92.71 101.6 0)
-			(hide yes)
-			(show_name no)
-			(do_not_autoplace no)
-			(effects
-				(font
-					(size 1.27 1.27)
-				)
-			)
-		)
-		(property "Datasheet" ""
-			(at 92.71 101.6 0)
-			(hide yes)
-			(show_name no)
-			(do_not_autoplace no)
-			(effects
-				(font
-					(size 1.27 1.27)
-				)
-			)
-		)
-		(property "Description" "Power symbol creates a global label with name \"GNDA\" , analog ground"
-			(at 92.71 101.6 0)
-			(hide yes)
-			(show_name no)
-			(do_not_autoplace no)
-			(effects
-				(font
-					(size 1.27 1.27)
-				)
-			)
-		)
-		(pin "1"
-		)
-		(instances
-			(project "Pico RP2350 USB Power"
-				(path "/f607a6cb-1f81-4ea5-ae65-67dd06ab9fb6"
-					(reference "#PWR043")
-					(unit 1)
-				)
-			)
-		)
-	)
-	(symbol
 		(lib_id "Connector_Generic_MountingPin:Conn_01x04_MountingPin")
 		(at 163.83 90.17 0)
@@
 	)
 	(symbol
-		(lib_id "power:GNDA")
-		(at 81.28 87.63 0)
-		(unit 1)
-		(body_style 1)
-		(exclude_from_sim no)
-		(in_bom yes)
-		(on_board yes)
-		(in_pos_files yes)
-		(dnp no)
-		(fields_autoplaced yes)
-		(property "Reference" "#PWR03"
-			(at 81.28 93.98 0)
-			(hide yes)
-			(show_name no)
-			(do_not_autoplace no)
-			(effects
-				(font
-					(size 1.27 1.27)
-				)
-			)
-		)
-		(property "Value" "GNDA"
-			(at 81.28 92.71 0)
-			(show_name no)
-			(do_not_autoplace no)
-			(effects
-				(font
-					(size 1.27 1.27)
-				)
-			)
-		)
-		(property "Footprint" ""
-			(at 81.28 87.63 0)
-			(hide yes)
-			(show_name no)
-			(do_not_autoplace no)
-			(effects
-				(font
-					(size 1.27 1.27)
-				)
-			)
-		)
-		(property "Datasheet" ""
-			(at 81.28 87.63 0)
-			(hide yes)
-			(show_name no)
-			(do_not_autoplace no)
-			(effects
-				(font
-					(size 1.27 1.27)
-				)
-			)
-		)
-		(property "Description" "Power symbol creates a global label with name \"GNDA\" , analog ground"
-			(at 81.28 87.63 0)
-			(hide yes)
-			(show_name no)
-			(do_not_autoplace no)
-			(effects
-				(font
-					(size 1.27 1.27)
-				)
-			)
-		)
-		(pin "1"
-		)
-		(instances
-			(project "Pico RP2350 USB Power"
-				(path "/f607a6cb-1f81-4ea5-ae65-67dd06ab9fb6"
-					(reference "#PWR03")
-					(unit 1)
-				)
-			)
-		)
-	)
-	(symbol
 		(lib_id "power:+5V")
 		(at 111.76 151.13 180)
@@
 	(symbol
 		(lib_id "power:GND")
-		(at 82.55 101.6 0)
+		(at 81.28 87.63 0)
 		(unit 1)
 		(body_style 1)
@@
 		(fields_autoplaced yes)
 		(property "Reference" "#PWR044"
-			(at 82.55 107.95 0)
+			(at 81.28 93.98 0)
 			(hide yes)
 			(show_name no)
@@
 		)
 		(property "Value" "GND"
-			(at 82.55 106.68 0)
+			(at 81.28 92.71 0)
 			(show_name no)
 			(do_not_autoplace no)
@@
 		)
 		(property "Footprint" ""
-			(at 82.55 101.6 0)
+			(at 81.28 87.63 0)
 			(hide yes)
 			(show_name no)
@@
 		)
 		(property "Datasheet" ""
-			(at 82.55 101.6 0)
+			(at 81.28 87.63 0)
 			(hide yes)
 			(show_name no)
@@
 		)
 		(property "Description" "Power symbol creates a global label with name \"GND\" , ground"
-			(at 82.55 101.6 0)
+			(at 81.28 87.63 0)
 			(hide yes)
 			(show_name no)
