File: electronics/scratch/IR Tester/IR Tester.kicad_sch (KiCad schematic)
At the start: 53 parts, among them J1 VS RAW, J10 IR TX AOE, J2 APA RAW, J3 XL RAW, Q3 AO3406, Q4 AO3406, Q5 AO3406, Q6 AO3406, U1 VSMB10940, U2 VSMB10940, U3 XL-3210IRC-940, U4 XL-3210IRC-940, U5 XL-1608UBC-06A, U6 XL-1608PGC-06

Commit message: IR tester board traced, parts assigned, sent to PCBWay
Parts:
- removed JP10, JP5, JP6, JP7, JP8, JP9: XL 21 T, Jumper:SolderJumper-2_P1.3mm_Bridged_Pad1.0x1.5mm, symbol Jumper:SolderJumper_2_Bridged
- removed LED10: XL-1608VRC-06, easyeda2kicad:LED0603-RD_PINK, symbol easyeda2kicad:XL-1608VRC-06
- removed LED11: P2-0603G1TS2-06T-002, easyeda2kicad:LED0603-RD_GREEN, symbol easyeda2kicad:F.0603.00025_P2-0603G1TS2-06T-002
- removed LED7: XL-1608SURC-06, easyeda2kicad:LED0603-RD_RED, symbol easyeda2kicad:XL-1608SURC-06
- removed LED8: XL-1608UGC-04, easyeda2kicad:LED0603-RD_GREEN, symbol easyeda2kicad:XL-1608UGC-04
- removed LED9: XL-1608UOC-06, easyeda2kicad:LED0603-R-RD_ORANGE, symbol easyeda2kicad:XL-1608UOC-06
- removed U5: XL-1608UBC-06A, easyeda2kicad:LED0603-R-RD, symbol easyeda2kicad:XL-1608UBC-06A
- removed U6: XL-1608PGC-06, easyeda2kicad:LED0603-RD_GREEN, symbol easyeda2kicad:XL-1608PGC-06
- removed VR1, VR3: 20K POT, easyeda2kicad:RES-ADJ-SMD_3P-L4.5-W4.5-P2.30-BL-FS, symbol easyeda2kicad:3314J-1-203E
- removed VR2, VR4, VR5, VR6: 10K POT, easyeda2kicad:RES-ADJ-SMD_3314J, symbol easyeda2kicad:3314J-1-103E
- added J4: Breakout Pins, Connector_PinHeader_2.54mm:PinHeader_1x06_P2.54mm_Vertical, symbol Connector:Conn_01x06_Pin
- J1, J10, J2, J3: now not fitted; now left out of the parts list
- Q3, Q4, Q5, Q6: LCSC Part (none) -> C42434120; MPN (none) -> AO3406(ES); Manufacturer (none) -> ElecSuper
- R10, R12, R13, R14, R16, R5, R7, R9: LCSC Part (none) -> C25612; MPN (none) -> 0805W8J0103T5E; Manufacturer (none) -> UNI-ROYAL
- R11: LCSC Part (none) -> C17622; MPN (none) -> 0805W8F300JT5E; Manufacturer (none) -> UNI-ROYAL
- R15: LCSC Part (none) -> C17408; MPN (none) -> 0805W8F1000T5E; Manufacturer (none) -> UNI-ROYAL
- R6: LCSC Part (none) -> C17561; MPN (none) -> 0805W8F220JT5E; Manufacturer (none) -> UNI-ROYAL
- R8: LCSC Part (none) -> C17679; MPN (none) -> 0805W8F402JT5E; Manufacturer (none) -> UNI-ROYAL
Connections:
- net +3.3V: now also J4.6 (Pin_6)
- net APA 50: now also J4.3 (Pin_3)
- net GND: now also J4.1 (Pin_1)
- net IR TX: now also J4.2 (Pin_2)
- net VS 65: now also J4.4 (Pin_4)
- net XL 21: now also J4.5 (Pin_5)
Other:
- note removed: "PUSH BUTTONS"
- note removed: "XINGLIGHT"
- moved on the sheet: JP1, JP2, JP3, JP4, LED2, LED4, LED5, LED6, R12, R13, R16, R9

Commit message: IR Tester - correct VSMB10940 polarity an amp circuit
Connections:
- net at Q5.3 (D): now also U1.2; no longer U1.3
- net at R11.2: now also U1.3; no longer U1.2
Other:
- title: (none) -> IR Tester
- moved on the sheet: R11
Changed lines of the file:
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@@
 	(generator_version "10.0")
 	(paper "A4")
+	(title_block
+		(title "IR Tester")
+		(date "2026-08-21")
+		(rev "b")
+	)
 	(rectangle
 		(start 80.01 13.97)
@@
 	(wire
 		(pts
-			(xy 44.45 104.14) (xy 53.34 104.14)
-		)
-		(stroke
-			(width 0)
-			(type default)
-		)
-	)
-	(wire
-		(pts
 			(xy 33.02 39.37) (xy 33.02 41.91)
 		)
@@
 	(wire
 		(pts
-			(xy 46.99 107.95) (xy 59.69 107.95)
+			(xy 46.99 105.41) (xy 66.04 105.41)
 		)
 		(stroke
@@
 	(wire
 		(pts
-			(xy 36.83 104.14) (xy 33.02 104.14)
-		)
-		(stroke
-			(width 0)
-			(type default)
-		)
-	)
-	(wire
-		(pts
-			(xy 59.69 107.95) (xy 59.69 110.49)
-		)
-		(stroke
-			(width 0)
-			(type default)
-		)
-	)
-	(wire
-		(pts
-			(xy 59.69 110.49) (xy 63.5 110.49)
+			(xy 71.12 119.38) (xy 74.93 119.38)
 		)
 		(stroke
@@
 	(wire
 		(pts
-			(xy 53.34 105.41) (xy 66.04 105.41)
+			(xy 93.98 39.37) (xy 104.14 39.37)
 		)
 		(stroke
@@
 	(wire
 		(pts
-			(xy 93.98 39.37) (xy 104.14 39.37)
+			(xy 46.99 66.04) (xy 53.34 66.04)
 		)
 		(stroke
@@
 	(wire
 		(pts
-			(xy 63.5 107.95) (xy 63.5 110.49)
+			(xy 71.12 64.77) (xy 71.12 69.85)
 		)
 		(stroke
@@
 	(wire
 		(pts
-			(xy 46.99 66.04) (xy 53.34 66.04)
+			(xy 95.25 67.31) (xy 100.33 67.31)
 		)
 		(stroke
@@
 	(wire
 		(pts
-			(xy 71.12 64.77) (xy 71.12 69.85)
+			(xy 87.63 109.22) (xy 95.25 109.22)
 		)
 		(stroke
@@
 	(wire
 		(pts
-			(xy 95.25 67.31) (xy 100.33 67.31)
+			(xy 60.96 119.38) (xy 60.96 107.95)
 		)
 		(stroke
@@
 	(wire
 		(pts
-			(xy 87.63 109.22) (xy 95.25 109.22)
+			(xy 166.37 77.47) (xy 171.45 77.47)
 		)
 		(stroke
@@
 	(wire
 		(pts
-			(xy 166.37 77.47) (xy 171.45 77.47)
+			(xy 45.72 24.13) (xy 50.8 24.13)
 		)
 		(stroke
@@
 	(wire
 		(pts
-			(xy 45.72 24.13) (xy 50.8 24.13)
+			(xy 93.98 29.21) (xy 104.14 29.21)
 		)
 		(stroke
@@
 	(wire
 		(pts
-			(xy 93.98 29.21) (xy 104.14 29.21)
+			(xy 46.99 105.41) (xy 46.99 107.95)
 		)
 		(stroke
@@
 	(wire
 		(pts
-			(xy 151.13 90.17) (xy 156.21 90.17)
+			(xy 60.96 107.95) (xy 66.04 107.95)
 		)
 		(stroke
@@
 	(wire
 		(pts
-			(xy 68.58 64.77) (xy 71.12 64.77)
+			(xy 151.13 90.17) (xy 156.21 90.17)
 		)
 		(stroke
@@
 	(wire
 		(pts
-			(xy 166.37 64.77) (xy 171.45 64.77)
+			(xy 68.58 64.77) (xy 71.12 64.77)
 		)
 		(stroke
@@
 	(wire
 		(pts
-			(xy 68.58 153.67) (xy 68.58 157.48)
+			(xy 166.37 64.77) (xy 171.45 64.77)
 		)
 		(stroke
@@
 	(wire
 		(pts
-			(xy 53.34 66.04) (xy 53.34 69.85)
+			(xy 68.58 153.67) (xy 68.58 157.48)
 		)
 		(stroke
@@
 	(wire
 		(pts
-			(xy 87.63 149.86) (xy 95.25 149.86)
+			(xy 53.34 66.04) (xy 53.34 69.85)
 		)
 		(stroke
@@
 	(wire
 		(pts
-			(xy 87.63 152.4) (xy 95.25 152.4)
+			(xy 87.63 149.86) (xy 95.25 149.86)
 		)
 		(stroke
@@
 	(wire
 		(pts
-			(xy 113.03 102.87) (xy 124.46 102.87)
+			(xy 87.63 152.4) (xy 95.25 152.4)
 		)
 		(stroke
@@
 	(wire
 		(pts
-			(xy 53.34 104.14) (xy 53.34 105.41)
+			(xy 113.03 102.87) (xy 124.46 102.87)
 		)
 		(stroke
@@
 	(wire
 		(pts
-			(xy 66.04 107.95) (xy 63.5 107.95)
-		)
-		(stroke
-			(width 0)
-			(type default)
-		)
-	)
-	(wire
-		(pts
 			(xy 87.63 67.31) (xy 92.71 67.31)
 		)
@@
 		)
 	)
+	(wire
+		(pts
+			(xy 63.5 119.38) (xy 60.96 119.38)
+		)
+		(stroke
+			(width 0)
+			(type default)
+		)
+	)
 	(label "VS 65"
 		(at 113.03 90.17 0)
@@
 	(symbol
 		(lib_id "power:VCC")
-		(at 33.02 104.14 0)
+		(at 74.93 119.38 0)
+		(mirror y)
 		(unit 1)
 		(body_style 1)
@@
 		(dnp no)
 		(property "Reference" "#PWR058"
-			(at 33.02 107.95 0)
+			(at 74.93 123.19 0)
 			(hide yes)
 			(show_name no)
@@
 		)
 		(property "Value" "+3.3V"
-			(at 33.02 100.33 0)
+			(at 74.93 115.57 0)
 			(show_name no)
 			(do_not_autoplace no)
@@
 		)
 		(property "Footprint" ""
-			(at 33.02 104.14 0)
+			(at 74.93 119.38 0)
 			(hide yes)
 			(show_name no)
@@
 		)
 		(property "Datasheet" ""
-			(at 33.02 104.14 0)
+			(at 74.93 119.38 0)
 			(hide yes)
 			(show_name no)
@@
 		)
 		(property "Description" "Power symbol creates a global label with name \"VCC\""
-			(at 33.02 104.14 0)
+			(at 74.93 119.38 0)
 			(hide yes)
 			(show_name no)
@@
 	(symbol
 		(lib_id "Device:R")
-		(at 40.64 104.14 90)
+		(at 67.31 119.38 270)
+		(mirror x)
 		(unit 1)
 		(body_style 1)
@@
 		(fields_autoplaced yes)
 		(property "Reference" "R11"
-			(at 40.64 97.79 90)
+			(at 67.31 113.03 90)
 			(show_name no)
 			(do_not_autoplace no)
@@
 		)
 		(property "Value" "30"
-			(at 40.64 100.33 90)
+			(at 67.31 115.57 90)
 			(show_name no)
 			(do_not_autoplace no)
@@
 		)
 		(property "Footprint" "Resistor_SMD:R_0805_2012Metric"
-			(at 40.64 105.918 90)
+			(at 67.31 121.158 90)
 			(hide yes)
 			(show_name no)
@@
 		)
 		(property "Datasheet" ""
-			(at 40.64 104.14 0)
+			(at 67.31 119.38 0)
 			(hide yes)
 			(show_name no)
@@
 		)
 		(property "Description" "Resistor"
-			(at 40.64 104.14 0)
+			(at 67.31 119.38 0)
 			(hide yes)
 			(show_name no)
@@
 		)
 		(property "LCSC Part" "C17622"
-			(at 40.64 104.14 90)
+			(at 67.31 119.38 90)
 			(hide yes)
 			(show_name no)
@@
 		)
 		(property "Manufacturer" "UNI-ROYAL"
-			(at -63.5 144.78 0)
+			(at 171.45 160.02 0)
 			(hide yes)
 			(show_name no)
@@
 		)
 		(property "MPN" "0805W8F300JT5E"
-			(at 40.64 104.14 90)
+			(at 67.31 119.38 90)
 			(hide yes)
 			(show_name no)
